Commit message: Launch File is done

File: install/bumperbot_description/share/bumperbot_description/urdf/bumperbot.urdf.xacro (robot description, xacro)
@@ -39,5 +39,5 @@
     </inertial-->
     <visual>
-      <origin xyz="0 0 0" rpy="0 0 0" />
+      <origin xyz="0 0 0" rpy="1.57 0 0" />
       <geometry>
         <mesh filename="package://bumperbot_description/meshes/wheel_right_link.STL" />
@@ -57,7 +57,7 @@
     <axis xyz="0 1 0" />
   </joint>
-  <!--link
+  <link
     name="wheel_left_link">
-    <inertial>
+    <!--inertial>
       <origin xyz="0 0.014 0" rpy="0 0 0" />
       <mass value="0.0530086043217644" />
@@ -65,5 +65,5 @@
                iyy="3.11510738759073E-05" iyz="-3.60499245082192E-10"
                izz="1.88266886146847E-05" />
-    </inertial>
+    </inertial-->
     <visual>
       <origin xyz="0 0 0" rpy="-1.57 0 0" />
@@ -72,10 +72,10 @@
       </geometry>
     </visual>
-    <collision>
+    <!--collision>
       <origin xyz="0 0.015 0" rpy="-1.57 0 0" />
       <geometry>
         <sphere radius="0.033"/>
       </geometry>
-    </collision>
+    </collision-->
   </link>
   <joint name="wheel_left_joint" type="continuous">
@@ -86,5 +86,5 @@
   </joint>
   <link name="caster_front_link">
-    <inertial>
+    <!--inertial>
       <origin xyz="3.89968128948481E-07 2.40073004698083E-07 0.00219173397061506" rpy="0 0 0" />
       <mass value="1.44379265037903E-06" />
@@ -92,5 +92,5 @@
                iyy="3.8713793085917E-11"  iyz="2.93909858781952E-15"
                izz="1.00967486676306E-10" />
-    </inertial>
+    </inertial-->
     <visual>
       <origin xyz="0 0 0" rpy="0 0 0" />
@@ -99,10 +99,10 @@
       </geometry>
     </visual>
-    <collision>
+    <!--collision>
       <origin xyz="0 0 0" rpy="0 0 0" />
       <geometry>
         <sphere radius="0.005"/>
       </geometry>
-    </collision>
+    </collision-->
   </link>
   <joint name="caster_front_joint" type="fixed">
@@ -113,5 +113,5 @@
   </joint>
   <link name="caster_rear_link">
-    <inertial>
+    <!--inertial>
       <origin xyz="3.8996812895542E-07 2.40073004698083E-07 0.00219173397061509" rpy="0 0 0" />
       <mass value="1.44379265037902E-06" />
@@ -119,5 +119,5 @@
                iyy="3.87137930859167E-11" iyz="2.939098587861E-15"
                izz="1.00967486676306E-10" />
-    </inertial>
+    </inertial-->
     <visual>
       <origin xyz="0 0 0" rpy="0 0 0" />
@@ -126,10 +126,10 @@
       </geometry>
     </visual>
-    <collision>
+    <!--collision>
       <origin xyz="0 0 0" rpy="0 0 0" />
       <geometry>
         <sphere radius="0.005"/>
       </geometry>
-    </collision>
+    </collision-->
   </link>
   <joint name="caster_rear_joint" type="fixed">
@@ -138,4 +138,4 @@
     <child link="caster_rear_link" />
     <axis xyz="0 0 0" />
-  </joint-->
+  </joint>
 </robot>

Commit message: Gazebo file with its launch file

File: install/bumperbot_description/share/bumperbot_description/urdf/bumperbot.urdf.xacro (robot description, xacro)
@@ -5,5 +5,5 @@
   <link name="base_footprint"/>
   <link name="base_link">
-    <!--inertial>
+    <inertial>
       <origin xyz="0 0 0.04" rpy="0.0 0.25 0.3" />
       <mass value="8.2573504e-01"/>
@@ -11,5 +11,5 @@
                iyy="2.1193702e-02" iyz="-5.0120904e-05"
                izz="2.0064271e-02" />
-    </inertial-->
+    </inertial>
     <visual>
       <origin rpy="0 0 0" xyz="0 0 0" />
@@ -18,10 +18,10 @@
       </geometry>
     </visual>
-    <!--collision>
+    <collision>
       <origin xyz="0 0 0" rpy="0 0 0" />
       <geometry>
         <mesh filename="package://bumperbot_description/meshes/base_link.STL" />
       </geometry>
-    </collision-->
+    </collision>
   </link>
   <joint name="base_joint" type="fixed">
@@ -31,5 +31,5 @@
   </joint>
   <link name="wheel_right_link">
-    <!--inertial>
+    <inertial>
       <origin xyz="0 -0.014 0" rpy="0 0 0" />
       <mass value="0.0530086090966721" />
@@ -37,5 +37,5 @@
                iyy="3.11510738647764E-05" iyz="-6.93560663069607E-11"
                izz="1.8801969558182E-05" />
-    </inertial-->
+    </inertial>
     <visual>
       <origin xyz="0 0 0" rpy="1.57 0 0" />
@@ -44,10 +44,10 @@
       </geometry>
     </visual>
-    <!--collision>
+    <collision>
       <origin xyz="0 -0.015 0" rpy="1.57 0 0" />
       <geometry>
         <sphere radius="0.033"/>
       </geometry>
-    </collision-->
+    </collision>
   </link>
   <joint name="wheel_right_joint" type="continuous">
@@ -59,5 +59,5 @@
   <link
     name="wheel_left_link">
-    <!--inertial>
+    <inertial>
       <origin xyz="0 0.014 0" rpy="0 0 0" />
       <mass value="0.0530086043217644" />
@@ -65,5 +65,5 @@
                iyy="3.11510738759073E-05" iyz="-3.60499245082192E-10"
                izz="1.88266886146847E-05" />
-    </inertial-->
+    </inertial>
     <visual>
       <origin xyz="0 0 0" rpy="-1.57 0 0" />
@@ -72,10 +72,10 @@
       </geometry>
     </visual>
-    <!--collision>
+    <collision>
       <origin xyz="0 0.015 0" rpy="-1.57 0 0" />
       <geometry>
         <sphere radius="0.033"/>
       </geometry>
-    </collision-->
+    </collision>
   </link>
   <joint name="wheel_left_joint" type="continuous">
@@ -86,5 +86,5 @@
   </joint>
   <link name="caster_front_link">
-    <!--inertial>
+    <inertial>
       <origin xyz="3.89968128948481E-07 2.40073004698083E-07 0.00219173397061506" rpy="0 0 0" />
       <mass value="1.44379265037903E-06" />
@@ -92,5 +92,5 @@
                iyy="3.8713793085917E-11"  iyz="2.93909858781952E-15"
                izz="1.00967486676306E-10" />
-    </inertial-->
+    </inertial>
     <visual>
       <origin xyz="0 0 0" rpy="0 0 0" />
@@ -99,10 +99,10 @@
       </geometry>
     </visual>
-    <!--collision>
+    <collision>
       <origin xyz="0 0 0" rpy="0 0 0" />
       <geometry>
         <sphere radius="0.005"/>
       </geometry>
-    </collision-->
+    </collision>
   </link>
   <joint name="caster_front_joint" type="fixed">
@@ -113,5 +113,5 @@
   </joint>
   <link name="caster_rear_link">
-    <!--inertial>
+    <inertial>
       <origin xyz="3.8996812895542E-07 2.40073004698083E-07 0.00219173397061509" rpy="0 0 0" />
       <mass value="1.44379265037902E-06" />
@@ -119,5 +119,5 @@
                iyy="3.87137930859167E-11" iyz="2.939098587861E-15"
                izz="1.00967486676306E-10" />
-    </inertial-->
+    </inertial>
     <visual>
       <origin xyz="0 0 0" rpy="0 0 0" />
@@ -126,10 +126,10 @@
       </geometry>
     </visual>
-    <!--collision>
+    <collision>
       <origin xyz="0 0 0" rpy="0 0 0" />
       <geometry>
         <sphere radius="0.005"/>
       </geometry>
-    </collision-->
+    </collision>
   </link>
   <joint name="caster_rear_joint" type="fixed">
@@ -139,3 +139,17 @@
     <axis xyz="0 0 0" />
   </joint>
+  <!--link name="can_link">
+    <visual>
+      <origin rpy="0 0 0" xyz="0 0 0" />
+      <geometry>
+        <mesh filename="package://bumperbot_description/meshes/can.STL" />
+      </geometry>
+    </visual>
+  </link>
+  <joint name="can_joint" type="fixed">
+    <origin xyz="-0.03 0.03 0.078" rpy="1.57 0 0" />
+    <parent link="base_link" />
+    <child link="can_link" />
+    <axis xyz="0 0 0" />
+  </joint-->
 </robot>

Commit message: Config & launch Control

File: install/bumperbot_description/share/bumperbot_description/urdf/bumperbot.urdf.xacro (robot description, xacro)
@@ -1,6 +1,8 @@
 <?xml version="1.0"?>
 <robot name="bumperbot" xmlns:xacro="http://ros.org/wiki/xacro">
-  <!-- Include Gazebo Parameters -->
-  <!--xacro:include filename="$(find bumperbot_description)/urdf/bumperbot_gazebo.xacro" /-->
+    <!-- Include Gazebo Parameters -->
+    <xacro:include filename="$(find bumperbot_description)/urdf/bumperbot_gazebo.xacro" />
+    <!-- Include ros2_control Plugins -->
+    <xacro:include filename="$(find bumperbot_description)/urdf/bumperbot_ros2_control.xacro" />
   <link name="base_footprint"/>
   <link name="base_link">

File: install/bumperbot_description/share/bumperbot_description/urdf/bumperbot_gazebo.xacro (robot description, xacro)
@@ -1,4 +1,18 @@
 <?xml version="1.0"?>
 <robot name="bumperbot" xmlns:xacro="http://ros.org/wiki/xacro">
+  <transmission name="wheel_right_transmission">
+    <plugin>transmission_interface/SimpleTransmission</plugin>
+    <actuator name="wheel_right_motor" role="actuator_right"/>
+    <joint name="wheel_right_joint"    role="joint_right">
+      <mechanical_reduction>1.0</mechanical_reduction>
+    </joint>
+  </transmission>
+  <transmission name="wheel_left_transmission">
+    <plugin>transmission_interface/SimpleTransmission</plugin>
+    <actuator name="wheel_left_motor" role="actuator_left"/>
+    <joint name="wheel_left_joint"    role="joint_left">
+      <mechanical_reduction>1.0</mechanical_reduction>
+    </joint>
+  </transmission>
   <!-- Wheels -->
   <gazebo reference="wheel_left_link">
@@ -37,3 +51,11 @@
     <maxVel>1.0</maxVel>
   </gazebo>
+  <!-- ROS 2 Control -->
+  <gazebo>
+    <plugin filename="libgazebo_ros2_control.so" name="gazebo_ros2_control">
+      <robot_param>robot_description</robot_param>
+      <robot_param_node>robot_state_publisher</robot_param_node>
+      <parameters>$(find bumperbot_controller)/config/bumperbot_controllers.yaml</parameters>
+    </plugin>
+  </gazebo>
 </robot>

Commit message: Proba & Sensor Fusion done!

File: install/bumperbot_description/share/bumperbot_description/urdf/bumperbot.urdf.xacro (robot description, xacro)
@@ -1,8 +1,8 @@
 <?xml version="1.0"?>
 <robot name="bumperbot" xmlns:xacro="http://ros.org/wiki/xacro">
-    <!-- Include Gazebo Parameters -->
-    <xacro:include filename="$(find bumperbot_description)/urdf/bumperbot_gazebo.xacro" />
-    <!-- Include ros2_control Plugins -->
-    <xacro:include filename="$(find bumperbot_description)/urdf/bumperbot_ros2_control.xacro" />
+  <!-- Include Gazebo Parameters -->
+  <xacro:include filename="$(find bumperbot_description)/urdf/bumperbot_gazebo.xacro" />
+  <!-- Include ros2_control Plugins -->
+  <xacro:include filename="$(find bumperbot_description)/urdf/bumperbot_ros2_control.xacro" />
   <link name="base_footprint"/>
   <link name="base_link">
@@ -15,5 +15,5 @@
     </inertial>
     <visual>
-      <origin rpy="0 0 0" xyz="0 0 0" />
+      <origin xyz="0 0 0" rpy="0 0 0" />
       <geometry>
         <mesh filename="package://bumperbot_description/meshes/base_link.STL" />
@@ -54,5 +54,5 @@
   </link>
   <joint name="wheel_right_joint" type="continuous">
-    <origin xyz="0 -0.07 0" rpy="0 0 0" />
+    <origin xyz="0 -0.0701101849418637 0" rpy="0 0 0" />
     <parent link="base_link" />
     <child link="wheel_right_link" />
@@ -141,17 +141,33 @@
     <axis xyz="0 0 0" />
   </joint>
-  <!--link name="can_link">
+  <link name="imu_link">
+    <inertial>
+      <origin xyz="-0.00552433659106688 0.000168210391520346 0.000514000497342681" rpy="0 0 0" />
+      <mass value="0.000528415362211671" />
+      <inertia ixx="1.46176048428261E-08" ixy="1.40015117949421E-10" ixz="-1.99633872937403E-12"
+               iyy="8.59662482954888E-09" iyz="7.52375112767959E-12"
+               izz="2.30279421279312E-08" />
+    </inertial>
     <visual>
-      <origin rpy="0 0 0" xyz="0 0 0" />
+      <origin xyz="0 0 0" rpy="0 0 0" />
       <geometry>
-        <mesh filename="package://bumperbot_description/meshes/can.STL" />
+        <mesh filename="package://bumperbot_description/meshes/imu_link.STL" />
       </geometry>
+      <material name="">
+        <color rgba="0.792156862745098 0.819607843137255 0.933333333333333 1" />
+      </material>
     </visual>
+    <collision>
+      <origin xyz="0 0 0" rpy="0 0 0" />
+      <geometry>
+        <mesh filename="package://bumperbot_description/meshes/imu_link.STL" />
+      </geometry>
+    </collision>
   </link>
-  <joint name="can_joint" type="fixed">
-    <origin xyz="-0.03 0.03 0.078" rpy="1.57 0 0" />
+  <joint name="imu_joint" type="fixed">
+    <origin xyz="0 0 0.0698986241758014" rpy="0 0 0" />
     <parent link="base_link" />
-    <child link="can_link" />
+    <child link="imu_link" />
     <axis xyz="0 0 0" />
-  </joint-->
+  </joint>
 </robot>

File: install/bumperbot_description/share/bumperbot_description/urdf/bumperbot_gazebo.xacro (robot description, xacro)
@@ -1,4 +1,5 @@
 <?xml version="1.0"?>
 <robot name="bumperbot" xmlns:xacro="http://ros.org/wiki/xacro">
+  <!-- Move this one to ros2 control -->
   <transmission name="wheel_right_transmission">
     <plugin>transmission_interface/SimpleTransmission</plugin>
@@ -59,3 +60,53 @@
     </plugin>
   </gazebo>
+  <!-- IMU -->
+  <gazebo reference="imu_link">
+    <sensor name="imu" type="imu">
+        <always_on>true</always_on>
+        <update_rate>100</update_rate>
+        <imu>
+          <angular_velocity>
+            <x>
+              <noise type="gaussian">
+                <mean>0.0</mean>
+                <stddev>2e-4</stddev>
+              </noise>
+            </x>
+            <y>
+              <noise type="gaussian">
+                <mean>0.0</mean>
+                <stddev>2e-4</stddev>
+              </noise>
+            </y>
+            <z>
+              <noise type="gaussian">
+                <mean>0.0</mean>
+                <stddev>2e-4</stddev>
+              </noise>
+            </z>
+          </angular_velocity>
+          <linear_acceleration>
+            <x>
+              <noise type="gaussian">
+                <mean>0.0</mean>
+                <stddev>1.7e-2</stddev>
+              </noise>
+            </x>
+            <y>
+              <noise type="gaussian">
+                <mean>0.0</mean>
+                <stddev>1.7e-2</stddev>
+              </noise>
+            </y>
+            <z>
+              <noise type="gaussian">
+                <mean>0.0</mean>
+                <stddev>1.7e-2</stddev>
+              </noise>
+            </z>
+          </linear_acceleration>
+        </imu>
+        <plugin name="imu" filename="libgazebo_ros_imu_sensor.so"/>
+    </sensor>
+  </gazebo>
 </robot>
